Commit message: Put seven capsules across the soles of lite_biped, lite and lite_pro
The biped shoe collided through 11 r8 spheres. They supported only 5% of
the underside of the shoe. A foot that fell with its side over a step
edge slid off and turned over in 40-42% of the drops, also with its
centre over the step, because the edge was between two spheres. lite and
lite_pro used two boxes from an older, shorter shoe.

The three variants now share one shoe: seven r8 capsules across the
sole, at equal intervals from the heel tip to the toe tip. The centres
of the capsule ends are on the sole outline. The five capsules under the
flat sole are flush with it, 65 mm below the foot origin, where the
training foot site is. The last two follow the toe spring. The MJCF
stage changes the scad cylinders into capsules.

Measured on lite_biped against the 11 spheres. Step time: mujoco-warp,
4096 worlds, the solver settings of the velocity task. Drops: a free
8 kg foot, 256 drops per case.

                                   spheres   7 capsules
  underside within 3 mm            5%        36%
  flat ground step time            -         +3 to +5%
  rough terrain step time          -         -23 to -25%
  stays on a step edge (side over
  the edge, centre over the step)  58-60%    97%
  lands turned over on bumps       12-14%    16-18%

The foot collisions of the URDF hub come from the new scad files,
without an Onshape export. The OpenSCAD parser of onshape-to-robot reads
each foot scad file, and a map from the part frame to the link frame
gives the URDF collisions. The map gives the old spheres and boxes, and
the new capsules, to 4 um. The MJCF and xacro of the three variants are
regenerated. Only the foot geoms change.

Co-Authored-By: Claude Opus 5.5 (1M context) <noreply@anthropic.com>
Claude-Session: https://claude.ai/code/session_01HpFUBhqSfbDuibPRVhscr9

File: lite_description/robots/lite/urdf/lite.urdf (robot description, URDF)
Before this commit: robot lite, 73 links, 72 joints
Links:
- link left_foot: geometry collision cylinder length=0.034 radius=0.008; collision cylinder length=0.048 radius=0.008
- link right_foot: geometry collision cylinder length=0.034 radius=0.008; collision cylinder length=0.048 radius=0.008

File: lite_description/robots/lite/xacro/lite.description.xacro (robot description, xacro)
@@ -162,13 +162,43 @@
       <!-- Part left_foot_parts -->
       <collision>
-        <origin xyz="0 0.05 0.015" rpy="1.5708 0 0" />
-        <geometry>
-          <box size="0.065 0.12 0.03" />
-        </geometry>
-      </collision>
-      <collision>
-        <origin xyz="0 0.04 0.11" rpy="1.91986 0 0" />
-        <geometry>
-          <box size="0.07 0.05 0.03" />
+        <origin xyz="-0.005 0.057 -0.056" rpy="1.5708 0 1.5708" />
+        <geometry>
+          <cylinder length="0.034" radius="0.008" />
+        </geometry>
+      </collision>
+      <collision>
+        <origin xyz="-0.0055 0.057 -0.0223" rpy="1.5708 0 1.5708" />
+        <geometry>
+          <cylinder length="0.067" radius="0.008" />
+        </geometry>
+      </collision>
+      <collision>
+        <origin xyz="-0.006 0.057 0.0113" rpy="1.5708 0 1.5708" />
+        <geometry>
+          <cylinder length="0.066" radius="0.008" />
+        </geometry>
+      </collision>
+      <collision>
+        <origin xyz="-0.0045 0.057 0.045" rpy="1.5708 0 1.5708" />
+        <geometry>
+          <cylinder length="0.071" radius="0.008" />
+        </geometry>
+      </collision>
+      <collision>
+        <origin xyz="-0.002 0.057 0.0787" rpy="1.5708 0 1.5708" />
+        <geometry>
+          <cylinder length="0.084" radius="0.008" />
+        </geometry>
+      </collision>
+      <collision>
+        <origin xyz="0.001 0.0526 0.1123" rpy="1.5708 0 1.5708" />
+        <geometry>
+          <cylinder length="0.082" radius="0.008" />
+        </geometry>
+      </collision>
+      <collision>
+        <origin xyz="0.004 0.0389 0.146" rpy="1.5708 0 1.5708" />
+        <geometry>
+          <cylinder length="0.048" radius="0.008" />
         </geometry>
       </collision>
@@ -375,13 +405,43 @@
       <!-- Part right_foot_parts -->
       <collision>
-        <origin xyz="0 0.05 0.015" rpy="1.5708 0 -0" />
-        <geometry>
-          <box size="0.065 0.12 0.03" />
-        </geometry>
-      </collision>
-      <collision>
-        <origin xyz="0 0.04 0.11" rpy="1.91986 0 -0" />
-        <geometry>
-          <box size="0.07 0.05 0.03" />
+        <origin xyz="0.005 0.057 -0.056" rpy="1.5708 0 1.5708" />
+        <geometry>
+          <cylinder length="0.034" radius="0.008" />
+        </geometry>
+      </collision>
+      <collision>
+        <origin xyz="0.0055 0.057 -0.0223" rpy="1.5708 0 1.5708" />
+        <geometry>
+          <cylinder length="0.067" radius="0.008" />
+        </geometry>
+      </collision>
+      <collision>
+        <origin xyz="0.006 0.057 0.0113" rpy="1.5708 0 1.5708" />
+        <geometry>
+          <cylinder length="0.066" radius="0.008" />
+        </geometry>
+      </collision>
+      <collision>
+        <origin xyz="0.0045 0.057 0.045" rpy="1.5708 0 1.5708" />
+        <geometry>
+          <cylinder length="0.071" radius="0.008" />
+        </geometry>
+      </collision>
+      <collision>
+        <origin xyz="0.002 0.057 0.0787" rpy="1.5708 0 1.5708" />
+        <geometry>
+          <cylinder length="0.084" radius="0.008" />
+        </geometry>
+      </collision>
+      <collision>
+        <origin xyz="-0.001 0.0526 0.1123" rpy="1.5708 0 1.5708" />
+        <geometry>
+          <cylinder length="0.082" radius="0.008" />
+        </geometry>
+      </collision>
+      <collision>
+        <origin xyz="-0.004 0.0389 0.146" rpy="1.5708 0 1.5708" />
+        <geometry>
+          <cylinder length="0.048" radius="0.008" />
         </geometry>
       </collision>

File: lite_description/robots/lite_biped/urdf/lite_biped.urdf (robot description, URDF)
Before this commit: robot lite_biped, 16 links, 15 joints
Links:
- link left_foot: geometry collision cylinder length=0.034 radius=0.008; collision cylinder length=0.048 radius=0.008
- link right_foot: geometry collision cylinder length=0.034 radius=0.008; collision cylinder length=0.048 radius=0.008

File: lite_description/robots/lite_biped/xacro/lite_biped.description.xacro (robot description, xacro)
@@ -171,67 +171,43 @@
       <!-- Part left_foot_parts -->
       <collision>
-        <origin xyz="-0.0046 0.057 -0.05998" rpy="1.5708 0 0" />
-        <geometry>
-          <sphere radius="0.008" />
-        </geometry>
-      </collision>
-      <collision>
-        <origin xyz="-0.03941 0.057 -0.0259" rpy="1.5708 0 0" />
-        <geometry>
-          <sphere radius="0.008" />
-        </geometry>
-      </collision>
-      <collision>
-        <origin xyz="0.02804 0.057 -0.02442" rpy="1.5708 0 0" />
-        <geometry>
-          <sphere radius="0.008" />
-        </geometry>
-      </collision>
-      <collision>
-        <origin xyz="-0.04209 0.057 0.02764" rpy="1.5708 0 0" />
-        <geometry>
-          <sphere radius="0.008" />
-        </geometry>
-      </collision>
-      <collision>
-        <origin xyz="0.03476 0.057 0.02877" rpy="1.5708 0 0" />
-        <geometry>
-          <sphere radius="0.008" />
-        </geometry>
-      </collision>
-      <collision>
-        <origin xyz="-0.04432 0.057 0.0812" rpy="1.5708 0 0" />
-        <geometry>
-          <sphere radius="0.008" />
-        </geometry>
-      </collision>
-      <collision>
-        <origin xyz="0.04148 0.057 0.08196" rpy="1.5708 0 0" />
-        <geometry>
-          <sphere radius="0.008" />
-        </geometry>
-      </collision>
-      <collision>
-        <origin xyz="-0.00047 0.057 0.09173" rpy="1.5708 0 0" />
-        <geometry>
-          <sphere radius="0.008" />
-        </geometry>
-      </collision>
-      <collision>
-        <origin xyz="-0.03438 0.04891 0.12489" rpy="1.5708 0 0" />
-        <geometry>
-          <sphere radius="0.008" />
-        </geometry>
-      </collision>
-      <collision>
-        <origin xyz="0.03932 0.04853 0.12597" rpy="1.5708 0 0" />
-        <geometry>
-          <sphere radius="0.008" />
-        </geometry>
-      </collision>
-      <collision>
-        <origin xyz="0.00465 0.03713 0.14874" rpy="1.5708 0 0" />
-        <geometry>
-          <sphere radius="0.008" />
+        <origin xyz="-0.005 0.057 -0.056" rpy="1.5708 0 1.5708" />
+        <geometry>
+          <cylinder length="0.034" radius="0.008" />
+        </geometry>
+      </collision>
+      <collision>
+        <origin xyz="-0.0055 0.057 -0.0223" rpy="1.5708 0 1.5708" />
+        <geometry>
+          <cylinder length="0.067" radius="0.008" />
+        </geometry>
+      </collision>
+      <collision>
+        <origin xyz="-0.006 0.057 0.0113" rpy="1.5708 0 1.5708" />
+        <geometry>
+          <cylinder length="0.066" radius="0.008" />
+        </geometry>
+      </collision>
+      <collision>
+        <origin xyz="-0.0045 0.057 0.045" rpy="1.5708 0 1.5708" />
+        <geometry>
+          <cylinder length="0.071" radius="0.008" />
+        </geometry>
+      </collision>
+      <collision>
+        <origin xyz="-0.002 0.057 0.0787" rpy="1.5708 0 1.5708" />
+        <geometry>
+          <cylinder length="0.084" radius="0.008" />
+        </geometry>
+      </collision>
+      <collision>
+        <origin xyz="0.001 0.0526 0.1123" rpy="1.5708 0 1.5708" />
+        <geometry>
+          <cylinder length="0.082" radius="0.008" />
+        </geometry>
+      </collision>
+      <collision>
+        <origin xyz="0.004 0.0389 0.146" rpy="1.5708 0 1.5708" />
+        <geometry>
+          <cylinder length="0.048" radius="0.008" />
         </geometry>
       </collision>
@@ -438,67 +414,43 @@
       <!-- Part right_foot_parts -->
       <collision>
-        <origin xyz="0.0046 0.057 -0.05998" rpy="1.5708 0 0" />
-        <geometry>
-          <sphere radius="0.008" />
-        </geometry>
-      </collision>
-      <collision>
-        <origin xyz="0.03941 0.057 -0.0259" rpy="1.5708 0 0" />
-        <geometry>
-          <sphere radius="0.008" />
-        </geometry>
-      </collision>
-      <collision>
-        <origin xyz="-0.02804 0.057 -0.02442" rpy="1.5708 0 0" />
-        <geometry>
-          <sphere radius="0.008" />
-        </geometry>
-      </collision>
-      <collision>
-        <origin xyz="0.04209 0.057 0.02764" rpy="1.5708 0 0" />
-        <geometry>
-          <sphere radius="0.008" />
-        </geometry>
-      </collision>
-      <collision>
-        <origin xyz="-0.03476 0.057 0.02877" rpy="1.5708 0 0" />
-        <geometry>
-          <sphere radius="0.008" />
-        </geometry>
-      </collision>
-      <collision>
-        <origin xyz="0.04432 0.057 0.0812" rpy="1.5708 0 0" />
-        <geometry>
-          <sphere radius="0.008" />
-        </geometry>
-      </collision>
-      <collision>
-        <origin xyz="-0.04148 0.057 0.08196" rpy="1.5708 0 0" />
-        <geometry>
-          <sphere radius="0.008" />
-        </geometry>
-      </collision>
-      <collision>
-        <origin xyz="0.00047 0.057 0.09173" rpy="1.5708 0 0" />
-        <geometry>
-          <sphere radius="0.008" />
-        </geometry>
-      </collision>
-      <collision>
-        <origin xyz="0.03438 0.04891 0.12489" rpy="1.5708 0 0" />
-        <geometry>
-          <sphere radius="0.008" />
-        </geometry>
-      </collision>
-      <collision>
-        <origin xyz="-0.03932 0.04853 0.12597" rpy="1.5708 0 0" />
-        <geometry>
-          <sphere radius="0.008" />
-        </geometry>
-      </collision>
-      <collision>
-        <origin xyz="-0.00465 0.03713 0.14874" rpy="1.5708 0 0" />
-        <geometry>
-          <sphere radius="0.008" />
+        <origin xyz="0.005 0.057 -0.056" rpy="1.5708 0 1.5708" />
+        <geometry>
+          <cylinder length="0.034" radius="0.008" />
+        </geometry>
+      </collision>
+      <collision>
+        <origin xyz="0.0055 0.057 -0.0223" rpy="1.5708 0 1.5708" />
+        <geometry>
+          <cylinder length="0.067" radius="0.008" />
+        </geometry>
+      </collision>
+      <collision>
+        <origin xyz="0.006 0.057 0.0113" rpy="1.5708 0 1.5708" />
+        <geometry>
+          <cylinder length="0.066" radius="0.008" />
+        </geometry>
+      </collision>
+      <collision>
+        <origin xyz="0.0045 0.057 0.045" rpy="1.5708 0 1.5708" />
+        <geometry>
+          <cylinder length="0.071" radius="0.008" />
+        </geometry>
+      </collision>
+      <collision>
+        <origin xyz="0.002 0.057 0.0787" rpy="1.5708 0 1.5708" />
+        <geometry>
+          <cylinder length="0.084" radius="0.008" />
+        </geometry>
+      </collision>
+      <collision>
+        <origin xyz="-0.001 0.0526 0.1123" rpy="1.5708 0 1.5708" />
+        <geometry>
+          <cylinder length="0.082" radius="0.008" />
+        </geometry>
+      </collision>
+      <collision>
+        <origin xyz="-0.004 0.0389 0.146" rpy="1.5708 0 1.5708" />
+        <geometry>
+          <cylinder length="0.048" radius="0.008" />
         </geometry>
       </collision>

File: lite_description/robots/lite_pro/urdf/lite_pro.urdf (robot description, URDF)
Before this commit: robot lite_pro, 75 links, 74 joints
Links:
- link left_foot: geometry collision cylinder length=0.034 radius=0.008; collision cylinder length=0.048 radius=0.008
- link right_foot: geometry collision cylinder length=0.034 radius=0.008; collision cylinder length=0.048 radius=0.008

File: lite_description/robots/lite_pro/xacro/lite_pro.description.xacro (robot description, xacro)
@@ -162,13 +162,43 @@
       <!-- Part left_foot_parts -->
       <collision>
-        <origin xyz="0 0.05 0.015" rpy="1.5708 0 0" />
-        <geometry>
-          <box size="0.065 0.12 0.03" />
-        </geometry>
-      </collision>
-      <collision>
-        <origin xyz="0 0.04 0.11" rpy="1.91986 0 0" />
-        <geometry>
-          <box size="0.07 0.05 0.03" />
+        <origin xyz="-0.005 0.057 -0.056" rpy="1.5708 0 1.5708" />
+        <geometry>
+          <cylinder length="0.034" radius="0.008" />
+        </geometry>
+      </collision>
+      <collision>
+        <origin xyz="-0.0055 0.057 -0.0223" rpy="1.5708 0 1.5708" />
+        <geometry>
+          <cylinder length="0.067" radius="0.008" />
+        </geometry>
+      </collision>
+      <collision>
+        <origin xyz="-0.006 0.057 0.0113" rpy="1.5708 0 1.5708" />
+        <geometry>
+          <cylinder length="0.066" radius="0.008" />
+        </geometry>
+      </collision>
+      <collision>
+        <origin xyz="-0.0045 0.057 0.045" rpy="1.5708 0 1.5708" />
+        <geometry>
+          <cylinder length="0.071" radius="0.008" />
+        </geometry>
+      </collision>
+      <collision>
+        <origin xyz="-0.002 0.057 0.0787" rpy="1.5708 0 1.5708" />
+        <geometry>
+          <cylinder length="0.084" radius="0.008" />
+        </geometry>
+      </collision>
+      <collision>
+        <origin xyz="0.001 0.0526 0.1123" rpy="1.5708 0 1.5708" />
+        <geometry>
+          <cylinder length="0.082" radius="0.008" />
+        </geometry>
+      </collision>
+      <collision>
+        <origin xyz="0.004 0.0389 0.146" rpy="1.5708 0 1.5708" />
+        <geometry>
+          <cylinder length="0.048" radius="0.008" />
         </geometry>
       </collision>
@@ -375,13 +405,43 @@
       <!-- Part right_foot_parts -->
       <collision>
-        <origin xyz="0 0.05 0.015" rpy="1.5708 0 -0" />
-        <geometry>
-          <box size="0.065 0.12 0.03" />
-        </geometry>
-      </collision>
-      <collision>
-        <origin xyz="0 0.04 0.11" rpy="1.91986 0 -0" />
-        <geometry>
-          <box size="0.07 0.05 0.03" />
+        <origin xyz="0.005 0.057 -0.056" rpy="1.5708 0 1.5708" />
+        <geometry>
+          <cylinder length="0.034" radius="0.008" />
+        </geometry>
+      </collision>
+      <collision>
+        <origin xyz="0.0055 0.057 -0.0223" rpy="1.5708 0 1.5708" />
+        <geometry>
+          <cylinder length="0.067" radius="0.008" />
+        </geometry>
+      </collision>
+      <collision>
+        <origin xyz="0.006 0.057 0.0113" rpy="1.5708 0 1.5708" />
+        <geometry>
+          <cylinder length="0.066" radius="0.008" />
+        </geometry>
+      </collision>
+      <collision>
+        <origin xyz="0.0045 0.057 0.045" rpy="1.5708 0 1.5708" />
+        <geometry>
+          <cylinder length="0.071" radius="0.008" />
+        </geometry>
+      </collision>
+      <collision>
+        <origin xyz="0.002 0.057 0.0787" rpy="1.5708 0 1.5708" />
+        <geometry>
+          <cylinder length="0.084" radius="0.008" />
+        </geometry>
+      </collision>
+      <collision>
+        <origin xyz="-0.001 0.0526 0.1123" rpy="1.5708 0 1.5708" />
+        <geometry>
+          <cylinder length="0.082" radius="0.008" />
+        </geometry>
+      </collision>
+      <collision>
+        <origin xyz="-0.004 0.0389 0.146" rpy="1.5708 0 1.5708" />
+        <geometry>
+          <cylinder length="0.048" radius="0.008" />
         </geometry>
       </collision>
