Commit message: Move the sole capsule ends 4 mm inside the shoe outline
The centres of the capsule ends were on the sole outline. Thus each
round end extended a full radius, 8 mm, past the shoe. Now the centres
are half a radius inside the outline. The ends extend 4 mm, and each
capsule is 8 mm shorter.

The flat sole goes to the outline. Thus on flat ground, the contact
points are now 4 mm inside the real sole edge on each side: 76 mm apart
at the widest capsule, against 84 mm of shoe. The narrower support has
an effect when the foot rolls. Drops of a free 8 kg foot, 256 drops per
case, against the capsules with their end centres on the outline:

                                   centres on   centres 4 mm
                                   outline      inside
  stays on a step edge (side over
  the edge, centre over the step)  97%          97%
  lands turned over on bumps       16-18%       23-24%
  roll pivot error vs the shell    1.6 mm       2.8 mm

Co-Authored-By: Claude Opus 5.5 (1M context) <noreply@anthropic.com>
Claude-Session: https://claude.ai/code/session_01HpFUBhqSfbDuibPRVhscr9

File: lite_description/robots/lite/urdf/lite.urdf (robot description, URDF)
Before this commit: robot lite, 73 links, 72 joints
Links:
- link left_foot: geometry collision cylinder length=0.026 radius=0.008; collision cylinder length=0.04 radius=0.008
- link right_foot: geometry collision cylinder length=0.026 radius=0.008; collision cylinder length=0.04 radius=0.008

File: lite_description/robots/lite/xacro/lite.description.xacro (robot description, xacro)
@@ -164,5 +164,5 @@
         <origin xyz="-0.005 0.057 -0.056" rpy="1.5708 0 1.5708" />
         <geometry>
-          <cylinder length="0.034" radius="0.008" />
+          <cylinder length="0.026" radius="0.008" />
         </geometry>
       </collision>
@@ -170,5 +170,5 @@
         <origin xyz="-0.0055 0.057 -0.0223" rpy="1.5708 0 1.5708" />
         <geometry>
-          <cylinder length="0.067" radius="0.008" />
+          <cylinder length="0.059" radius="0.008" />
         </geometry>
       </collision>
@@ -176,5 +176,5 @@
         <origin xyz="-0.006 0.057 0.0113" rpy="1.5708 0 1.5708" />
         <geometry>
-          <cylinder length="0.066" radius="0.008" />
+          <cylinder length="0.058" radius="0.008" />
         </geometry>
       </collision>
@@ -182,5 +182,5 @@
         <origin xyz="-0.0045 0.057 0.045" rpy="1.5708 0 1.5708" />
         <geometry>
-          <cylinder length="0.071" radius="0.008" />
+          <cylinder length="0.063" radius="0.008" />
         </geometry>
       </collision>
@@ -188,5 +188,5 @@
         <origin xyz="-0.002 0.057 0.0787" rpy="1.5708 0 1.5708" />
         <geometry>
-          <cylinder length="0.084" radius="0.008" />
+          <cylinder length="0.076" radius="0.008" />
         </geometry>
       </collision>
@@ -194,5 +194,5 @@
         <origin xyz="0.001 0.0526 0.1123" rpy="1.5708 0 1.5708" />
         <geometry>
-          <cylinder length="0.082" radius="0.008" />
+          <cylinder length="0.074" radius="0.008" />
         </geometry>
       </collision>
@@ -200,5 +200,5 @@
         <origin xyz="0.004 0.0389 0.146" rpy="1.5708 0 1.5708" />
         <geometry>
-          <cylinder length="0.048" radius="0.008" />
+          <cylinder length="0.04" radius="0.008" />
         </geometry>
       </collision>
@@ -407,5 +407,5 @@
         <origin xyz="0.005 0.057 -0.056" rpy="1.5708 0 1.5708" />
         <geometry>
-          <cylinder length="0.034" radius="0.008" />
+          <cylinder length="0.026" radius="0.008" />
         </geometry>
       </collision>
@@ -413,5 +413,5 @@
         <origin xyz="0.0055 0.057 -0.0223" rpy="1.5708 0 1.5708" />
         <geometry>
-          <cylinder length="0.067" radius="0.008" />
+          <cylinder length="0.059" radius="0.008" />
         </geometry>
       </collision>
@@ -419,5 +419,5 @@
         <origin xyz="0.006 0.057 0.0113" rpy="1.5708 0 1.5708" />
         <geometry>
-          <cylinder length="0.066" radius="0.008" />
+          <cylinder length="0.058" radius="0.008" />
         </geometry>
       </collision>
@@ -425,5 +425,5 @@
         <origin xyz="0.0045 0.057 0.045" rpy="1.5708 0 1.5708" />
         <geometry>
-          <cylinder length="0.071" radius="0.008" />
+          <cylinder length="0.063" radius="0.008" />
         </geometry>
       </collision>
@@ -431,5 +431,5 @@
         <origin xyz="0.002 0.057 0.0787" rpy="1.5708 0 1.5708" />
         <geometry>
-          <cylinder length="0.084" radius="0.008" />
+          <cylinder length="0.076" radius="0.008" />
         </geometry>
       </collision>
@@ -437,5 +437,5 @@
         <origin xyz="-0.001 0.0526 0.1123" rpy="1.5708 0 1.5708" />
         <geometry>
-          <cylinder length="0.082" radius="0.008" />
+          <cylinder length="0.074" radius="0.008" />
         </geometry>
       </collision>
@@ -443,5 +443,5 @@
         <origin xyz="-0.004 0.0389 0.146" rpy="1.5708 0 1.5708" />
         <geometry>
-          <cylinder length="0.048" radius="0.008" />
+          <cylinder length="0.04" radius="0.008" />
         </geometry>
       </collision>

File: lite_description/robots/lite_biped/urdf/lite_biped.urdf (robot description, URDF)
Before this commit: robot lite_biped, 16 links, 15 joints
Links:
- link left_foot: geometry collision cylinder length=0.026 radius=0.008; collision cylinder length=0.04 radius=0.008
- link right_foot: geometry collision cylinder length=0.026 radius=0.008; collision cylinder length=0.04 radius=0.008

File: lite_description/robots/lite_biped/xacro/lite_biped.description.xacro (robot description, xacro)
@@ -173,5 +173,5 @@
         <origin xyz="-0.005 0.057 -0.056" rpy="1.5708 0 1.5708" />
         <geometry>
-          <cylinder length="0.034" radius="0.008" />
+          <cylinder length="0.026" radius="0.008" />
         </geometry>
       </collision>
@@ -179,5 +179,5 @@
         <origin xyz="-0.0055 0.057 -0.0223" rpy="1.5708 0 1.5708" />
         <geometry>
-          <cylinder length="0.067" radius="0.008" />
+          <cylinder length="0.059" radius="0.008" />
         </geometry>
       </collision>
@@ -185,5 +185,5 @@
         <origin xyz="-0.006 0.057 0.0113" rpy="1.5708 0 1.5708" />
         <geometry>
-          <cylinder length="0.066" radius="0.008" />
+          <cylinder length="0.058" radius="0.008" />
         </geometry>
       </collision>
@@ -191,5 +191,5 @@
         <origin xyz="-0.0045 0.057 0.045" rpy="1.5708 0 1.5708" />
         <geometry>
-          <cylinder length="0.071" radius="0.008" />
+          <cylinder length="0.063" radius="0.008" />
         </geometry>
       </collision>
@@ -197,5 +197,5 @@
         <origin xyz="-0.002 0.057 0.0787" rpy="1.5708 0 1.5708" />
         <geometry>
-          <cylinder length="0.084" radius="0.008" />
+          <cylinder length="0.076" radius="0.008" />
         </geometry>
       </collision>
@@ -203,5 +203,5 @@
         <origin xyz="0.001 0.0526 0.1123" rpy="1.5708 0 1.5708" />
         <geometry>
-          <cylinder length="0.082" radius="0.008" />
+          <cylinder length="0.074" radius="0.008" />
         </geometry>
       </collision>
@@ -209,5 +209,5 @@
         <origin xyz="0.004 0.0389 0.146" rpy="1.5708 0 1.5708" />
         <geometry>
-          <cylinder length="0.048" radius="0.008" />
+          <cylinder length="0.04" radius="0.008" />
         </geometry>
       </collision>
@@ -416,5 +416,5 @@
         <origin xyz="0.005 0.057 -0.056" rpy="1.5708 0 1.5708" />
         <geometry>
-          <cylinder length="0.034" radius="0.008" />
+          <cylinder length="0.026" radius="0.008" />
         </geometry>
       </collision>
@@ -422,5 +422,5 @@
         <origin xyz="0.0055 0.057 -0.0223" rpy="1.5708 0 1.5708" />
         <geometry>
-          <cylinder length="0.067" radius="0.008" />
+          <cylinder length="0.059" radius="0.008" />
         </geometry>
       </collision>
@@ -428,5 +428,5 @@
         <origin xyz="0.006 0.057 0.0113" rpy="1.5708 0 1.5708" />
         <geometry>
-          <cylinder length="0.066" radius="0.008" />
+          <cylinder length="0.058" radius="0.008" />
         </geometry>
       </collision>
@@ -434,5 +434,5 @@
         <origin xyz="0.0045 0.057 0.045" rpy="1.5708 0 1.5708" />
         <geometry>
-          <cylinder length="0.071" radius="0.008" />
+          <cylinder length="0.063" radius="0.008" />
         </geometry>
       </collision>
@@ -440,5 +440,5 @@
         <origin xyz="0.002 0.057 0.0787" rpy="1.5708 0 1.5708" />
         <geometry>
-          <cylinder length="0.084" radius="0.008" />
+          <cylinder length="0.076" radius="0.008" />
         </geometry>
       </collision>
@@ -446,5 +446,5 @@
         <origin xyz="-0.001 0.0526 0.1123" rpy="1.5708 0 1.5708" />
         <geometry>
-          <cylinder length="0.082" radius="0.008" />
+          <cylinder length="0.074" radius="0.008" />
         </geometry>
       </collision>
@@ -452,5 +452,5 @@
         <origin xyz="-0.004 0.0389 0.146" rpy="1.5708 0 1.5708" />
         <geometry>
-          <cylinder length="0.048" radius="0.008" />
+          <cylinder length="0.04" radius="0.008" />
         </geometry>
       </collision>

File: lite_description/robots/lite_pro/urdf/lite_pro.urdf (robot description, URDF)
Before this commit: robot lite_pro, 75 links, 74 joints
Links:
- link left_foot: geometry collision cylinder length=0.026 radius=0.008; collision cylinder length=0.04 radius=0.008
- link right_foot: geometry collision cylinder length=0.026 radius=0.008; collision cylinder length=0.04 radius=0.008

File: lite_description/robots/lite_pro/xacro/lite_pro.description.xacro (robot description, xacro)
@@ -164,5 +164,5 @@
         <origin xyz="-0.005 0.057 -0.056" rpy="1.5708 0 1.5708" />
         <geometry>
-          <cylinder length="0.034" radius="0.008" />
+          <cylinder length="0.026" radius="0.008" />
         </geometry>
       </collision>
@@ -170,5 +170,5 @@
         <origin xyz="-0.0055 0.057 -0.0223" rpy="1.5708 0 1.5708" />
         <geometry>
-          <cylinder length="0.067" radius="0.008" />
+          <cylinder length="0.059" radius="0.008" />
         </geometry>
       </collision>
@@ -176,5 +176,5 @@
         <origin xyz="-0.006 0.057 0.0113" rpy="1.5708 0 1.5708" />
         <geometry>
-          <cylinder length="0.066" radius="0.008" />
+          <cylinder length="0.058" radius="0.008" />
         </geometry>
       </collision>
@@ -182,5 +182,5 @@
         <origin xyz="-0.0045 0.057 0.045" rpy="1.5708 0 1.5708" />
         <geometry>
-          <cylinder length="0.071" radius="0.008" />
+          <cylinder length="0.063" radius="0.008" />
         </geometry>
       </collision>
@@ -188,5 +188,5 @@
         <origin xyz="-0.002 0.057 0.0787" rpy="1.5708 0 1.5708" />
         <geometry>
-          <cylinder length="0.084" radius="0.008" />
+          <cylinder length="0.076" radius="0.008" />
         </geometry>
       </collision>
@@ -194,5 +194,5 @@
         <origin xyz="0.001 0.0526 0.1123" rpy="1.5708 0 1.5708" />
         <geometry>
-          <cylinder length="0.082" radius="0.008" />
+          <cylinder length="0.074" radius="0.008" />
         </geometry>
       </collision>
@@ -200,5 +200,5 @@
         <origin xyz="0.004 0.0389 0.146" rpy="1.5708 0 1.5708" />
         <geometry>
-          <cylinder length="0.048" radius="0.008" />
+          <cylinder length="0.04" radius="0.008" />
         </geometry>
       </collision>
@@ -407,5 +407,5 @@
         <origin xyz="0.005 0.057 -0.056" rpy="1.5708 0 1.5708" />
         <geometry>
-          <cylinder length="0.034" radius="0.008" />
+          <cylinder length="0.026" radius="0.008" />
         </geometry>
       </collision>
@@ -413,5 +413,5 @@
         <origin xyz="0.0055 0.057 -0.0223" rpy="1.5708 0 1.5708" />
         <geometry>
-          <cylinder length="0.067" radius="0.008" />
+          <cylinder length="0.059" radius="0.008" />
         </geometry>
       </collision>
@@ -419,5 +419,5 @@
         <origin xyz="0.006 0.057 0.0113" rpy="1.5708 0 1.5708" />
         <geometry>
-          <cylinder length="0.066" radius="0.008" />
+          <cylinder length="0.058" radius="0.008" />
         </geometry>
       </collision>
@@ -425,5 +425,5 @@
         <origin xyz="0.0045 0.057 0.045" rpy="1.5708 0 1.5708" />
         <geometry>
-          <cylinder length="0.071" radius="0.008" />
+          <cylinder length="0.063" radius="0.008" />
         </geometry>
       </collision>
@@ -431,5 +431,5 @@
         <origin xyz="0.002 0.057 0.0787" rpy="1.5708 0 1.5708" />
         <geometry>
-          <cylinder length="0.084" radius="0.008" />
+          <cylinder length="0.076" radius="0.008" />
         </geometry>
       </collision>
@@ -437,5 +437,5 @@
         <origin xyz="-0.001 0.0526 0.1123" rpy="1.5708 0 1.5708" />
         <geometry>
-          <cylinder length="0.082" radius="0.008" />
+          <cylinder length="0.074" radius="0.008" />
         </geometry>
       </collision>
@@ -443,5 +443,5 @@
         <origin xyz="-0.004 0.0389 0.146" rpy="1.5708 0 1.5708" />
         <geometry>
-          <cylinder length="0.048" radius="0.008" />
+          <cylinder length="0.04" radius="0.008" />
         </geometry>
       </collision>
